File: Microcontroller Draft/Output Logic.sch (EAGLE design)
At the start: 4 parts, among them IC1 74HC86N, T1 BSS110, T2 BSS110, T3 BSS110

Commit message: Added a truth table to the output logic schematic
Other:
- note added: "Truth Table P1 | P2 | O H L T1 L H T2 L L T3"
Changed lines of the file:
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@@
 T2 = 7805 Transistor
 T3 = LD33V Transistor</text>
+<text x="83.82" y="48.26" size="1.778" layer="91">Truth Table
+P1 | P2 | O
+ H    L     T1
+ L    H     T2
+ L    L      T3</text>
 </plain>
 <instances>
