File: Microcontroller Draft/Microcontroller.sch (EAGLE design)
At the start: 6 parts, among them IC1 7805T

Commit message: Added the rotary encoder to the mix
Connections:
- net ROT_A renamed RE_A
- net ROT_B renamed RE_B
Changed lines of the file:
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@@
 </segment>
 </net>
-<net name="ROT_A" class="0">
+<net name="RE_A" class="0">
 <segment>
 <pinref part="U$1" gate="G$1" pin="15"/>
@@
 </segment>
 </net>
-<net name="ROT_B" class="0">
+<net name="RE_B" class="0">
 <segment>
 <pinref part="U$1" gate="G$1" pin="18"/>
