File: Revision A.sch (EAGLE design)
At the start: 51 parts, among them IC1 7805T, Q1 IRF9530, Q2 IRF9530, Q3 IRF9530, T1 BC547, T2 BC547, T3 BC547, U1 TLV2372IP, U2 LCD-16X2SILK

Commit message: Added the input barrel jack
Parts:
- added J1: POWER_JACKPTH, SparkFun-Connectors:POWER_JACKPTH
Connections:
- net GND: now also J1.GND
- net VIN: now also J1.PWR
Changed lines of the file:
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@@
 <layers>
 <layer number="1" name="Top" color="4" fill="1" visible="no" active="no"/>
+<layer number="2" name="Route2" color="1" fill="3" visible="no" active="no"/>
+<layer number="3" name="Route3" color="4" fill="3" visible="no" active="no"/>
+<layer number="14" name="Route14" color="1" fill="6" visible="no" active="no"/>
+<layer number="15" name="Route15" color="4" fill="6" visible="no" active="no"/>
 <layer number="16" name="Bottom" color="1" fill="1" visible="no" active="no"/>
 <layer number="17" name="Pads" color="2" fill="1" visible="no" active="no"/>
@@
 <part name="RE1" library="Custom Stuff" deviceset="ECW1J-B24-BCCO24L" device="ECW1J-B"/>
 <part name="P+10" library="supply1" deviceset="+5V" device=""/>
+<part name="J1" library="SparkFun-Connectors" deviceset="POWER_JACK" device="PTH"/>
+<part name="SUPPLY12" library="supply2" deviceset="GND" device=""/>
 </parts>
 <sheets>
@@
 <instance part="RE1" gate="G$1" x="114.3" y="175.26"/>
 <instance part="P+10" gate="1" x="124.46" y="165.1"/>
+<instance part="J1" gate="G$1" x="177.8" y="170.18"/>
+<instance part="SUPPLY12" gate="GND" x="190.5" y="162.56"/>
 </instances>
 <busses>
@@
 <wire x1="0" y1="177.8" x2="10.16" y2="177.8" width="0.1524" layer="91"/>
 <junction x="10.16" y="177.8"/>
+</segment>
+<segment>
+<pinref part="J1" gate="G$1" pin="GND"/>
+<wire x1="180.34" y1="172.72" x2="190.5" y2="172.72" width="0.1524" layer="91"/>
+<wire x1="190.5" y1="172.72" x2="190.5" y2="165.1" width="0.1524" layer="91"/>
+<pinref part="SUPPLY12" gate="GND" pin="GND"/>
 </segment>
 </net>
@@
 <label x="581.66" y="208.28" size="1.778" layer="95"/>
 </segment>
+<segment>
+<pinref part="J1" gate="G$1" pin="PWR"/>
+<wire x1="180.34" y1="177.8" x2="190.5" y2="177.8" width="0.1524" layer="91"/>
+<wire x1="190.5" y1="177.8" x2="190.5" y2="187.96" width="0.1524" layer="91"/>
+<label x="187.96" y="187.96" size="1.778" layer="95"/>
+</segment>
 </net>

Commit message: Fixed the RESET pin connection
Connections:
- net +5V: now also R2.2; no longer S_RST.P
- net GND: now also S_RST.P; no longer R2.2
Changed lines of the file:
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@@
 <instance part="SUPPLY4" gate="GND" x="320.04" y="73.66"/>
 <instance part="P+4" gate="1" x="320.04" y="91.44"/>
-<instance part="SUPPLY5" gate="GND" x="284.48" y="73.66"/>
+<instance part="SUPPLY5" gate="GND" x="274.32" y="93.98"/>
 <instance part="R2" gate="G$1" x="292.1" y="83.82" rot="R180"/>
 <instance part="S_RST" gate="1" x="289.56" y="104.14" rot="R270"/>
-<instance part="P+5" gate="1" x="274.32" y="114.3"/>
+<instance part="P+5" gate="1" x="284.48" y="96.52"/>
 <instance part="R1" gate="R?" x="246.38" y="152.4"/>
 <instance part="SUPPLY6" gate="GND" x="241.3" y="165.1"/>
@@
 </segment>
 <segment>
-<pinref part="S_RST" gate="1" pin="P"/>
-<pinref part="P+5" gate="1" pin="+5V"/>
-<wire x1="284.48" y1="104.14" x2="274.32" y2="104.14" width="0.1524" layer="91"/>
-<wire x1="274.32" y1="104.14" x2="274.32" y2="111.76" width="0.1524" layer="91"/>
-</segment>
-<segment>
 <wire x1="243.84" y1="185.42" x2="243.84" y2="177.8" width="0.1524" layer="91"/>
 <pinref part="P+6" gate="1" pin="+5V"/>
@@
 <wire x1="124.46" y1="157.48" x2="124.46" y2="162.56" width="0.1524" layer="91"/>
 </segment>
+<segment>
+<pinref part="R2" gate="G$1" pin="2"/>
+<wire x1="287.02" y1="83.82" x2="284.48" y2="83.82" width="0.1524" layer="91"/>
+<pinref part="P+5" gate="1" pin="+5V"/>
+<wire x1="284.48" y1="83.82" x2="284.48" y2="93.98" width="0.1524" layer="91"/>
+</segment>
 </net>
 <net name="GND" class="0">
@@
 <wire x1="312.42" y1="81.28" x2="320.04" y2="81.28" width="0.1524" layer="91"/>
 <wire x1="320.04" y1="81.28" x2="320.04" y2="76.2" width="0.1524" layer="91"/>
-</segment>
-<segment>
-<pinref part="R2" gate="G$1" pin="2"/>
-<pinref part="SUPPLY5" gate="GND" pin="GND"/>
-<wire x1="287.02" y1="83.82" x2="284.48" y2="83.82" width="0.1524" layer="91"/>
-<wire x1="284.48" y1="83.82" x2="284.48" y2="76.2" width="0.1524" layer="91"/>
 </segment>
 <segment>
@@
 <pinref part="SUPPLY12" gate="GND" pin="GND"/>
 </segment>
+<segment>
+<pinref part="S_RST" gate="1" pin="P"/>
+<wire x1="284.48" y1="104.14" x2="274.32" y2="104.14" width="0.1524" layer="91"/>
+<pinref part="SUPPLY5" gate="GND" pin="GND"/>
+<wire x1="274.32" y1="104.14" x2="274.32" y2="96.52" width="0.1524" layer="91"/>
+</segment>
 </net>

Commit message: Fixed the voltage regulator for the MCU
Parts:
- removed IC1: 7805T, linear:7805T
- added IC2: LD117AV33, v-reg:LD117AV33
Connections:
- net +5V: now also IC2.OUT; no longer IC1.VO
- net GND: now also IC2.ADJ; no longer IC1.GND
- net VIN: now also IC2.IN; no longer IC1.VI
Changed lines of the file:
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@@
 <part name="SUPPLY1" library="supply2" deviceset="GND" device=""/>
 <part name="U$1" library="TI_MSP430_v16" deviceset="G2XX3---N20" device=""/>
-<part name="IC1" library="linear" deviceset="78*" device="T" technology="05"/>
 <part name="SUPPLY2" library="supply2" deviceset="GND" device=""/>
 <part name="P+2" library="supply1" deviceset="+5V" device=""/>
@@
 <part name="J1" library="SparkFun-Connectors" deviceset="POWER_JACK" device="PTH"/>
 <part name="SUPPLY12" library="supply2" deviceset="GND" device=""/>
+<part name="IC2" library="v-reg" deviceset="LD117A?*" device="V" technology="33"/>
 </parts>
 <sheets>
@@
 <instance part="SUPPLY1" gate="GND" x="254" y="40.64"/>
 <instance part="U$1" gate="G$1" x="200.66" y="73.66"/>
-<instance part="IC1" gate="A1" x="200.66" y="134.62"/>
 <instance part="SUPPLY2" gate="GND" x="200.66" y="121.92"/>
 <instance part="P+2" gate="1" x="215.9" y="142.24"/>
@@
 <instance part="J1" gate="G$1" x="177.8" y="170.18"/>
 <instance part="SUPPLY12" gate="GND" x="190.5" y="162.56"/>
+<instance part="IC2" gate="G$1" x="200.66" y="134.62"/>
 </instances>
 <busses>
@@
 </segment>
 <segment>
-<pinref part="IC1" gate="A1" pin="VO"/>
-<wire x1="210.82" y1="134.62" x2="215.9" y2="134.62" width="0.1524" layer="91"/>
+<wire x1="208.28" y1="134.62" x2="215.9" y2="134.62" width="0.1524" layer="91"/>
 <wire x1="215.9" y1="134.62" x2="215.9" y2="139.7" width="0.1524" layer="91"/>
 <pinref part="P+2" gate="1" pin="+5V"/>
+<pinref part="IC2" gate="G$1" pin="OUT"/>
 </segment>
 <segment>
@@
 </segment>
 <segment>
-<pinref part="IC1" gate="A1" pin="GND"/>
 <pinref part="SUPPLY2" gate="GND" pin="GND"/>
 <wire x1="200.66" y1="127" x2="200.66" y2="124.46" width="0.1524" layer="91"/>
+<pinref part="IC2" gate="G$1" pin="ADJ"/>
 </segment>
 <segment>
@@
 <net name="VIN" class="0">
 <segment>
-<pinref part="IC1" gate="A1" pin="VI"/>
-<wire x1="190.5" y1="134.62" x2="185.42" y2="134.62" width="0.1524" layer="91"/>
+<wire x1="193.04" y1="134.62" x2="185.42" y2="134.62" width="0.1524" layer="91"/>
 <wire x1="185.42" y1="134.62" x2="185.42" y2="139.7" width="0.1524" layer="91"/>
 <label x="182.88" y="139.7" size="1.778" layer="95"/>
-</segment>
-<segment>
+<pinref part="IC2" gate="G$1" pin="IN"/>
+</segment>
+<segment>
