File: Mini Rev B/Mini Power Supply.brd (EAGLE design)
At the start: 52.1 x 36.8 mm, 23 parts, among them Q1 BC817-25LT1SMD

Commit message: Finished the negative rail
Parts:
- removed IADJ: (no value), v-reg:317TS
- removed Q1: BC817-25LT1SMD, transistor-npn:SOT23-BEC
- removed R5, R6: 100Ω, rcl:R0805
- removed VIN_SEL: (no value), pinhead:2X02
- added -I_PRB: (no value), pinhead:1X02
- added -OUTPUT: M02JST-PTH-2, SparkFun-Connectors:JST-2-PTH
- added C4: 0.1uF, rcl:C0805
- added C6: 10uF, rcl:E2,5-6
- added C7: 1uF, rcl:E2,5-6
- added D4, D5: (no value), diode:SOD323-W
- added ON-: (no value), led:CHIPLED_1206
- added SW_N, SW_P: (no value), SparkFun-Electromechanical:SWITCH-SPDT_LOCK.007S
- added VADJ1: (no value), v-reg:317TS
- R1: value 560Ω -> 240Ω
- R2: value TRIMPOT-PTH-KNOB -> 240Ω; device SparkFun-Electromechanical:3386U -> rcl:R0805
- R3: value TRIMPOT-PTH-KNOB -> 5kΩ; device SparkFun-Electromechanical:3386U -> bourns:3386W
- R4: value 100Ω -> 5kΩ; device rcl:R0805 -> bourns:3386W
- moved R8 107.6 mm to (-20.3, -88.9), turned to 0 degrees
- moved R2 65.2 mm to (-8.89, -48.3)
- moved R4 42.3 mm to (-6.35, -25.4)
- moved R3 25.0 mm to (-6.35, -15.2)
- renumbered I_PRB to +I_PRB, ON to ON+, OUTPUT to +OUTPUT
Connections:
- removed net IADJ_IN: IADJ.3, VIN_SEL.2
- removed net N$8: Q1.B, R8.2
- removed net VADJ_IN: C1.1, D2.C, IADJ.1, R3.3, R6.1, VADJ.3, VIN_SEL.4
- removed net VOUT: +I_PRB.1, C2.+, D1.C, D2.A, R1.2, R8.1, VADJ.2
- new net +VOUT: +I_PRB.1, C2.+, D1.C, D2.A, R1.2, VADJ.2
- new net -VOUT: -I_PRB.1, C6.-, D4.C, D5.A, R2.2, VADJ1.2
- new net N$10: -I_PRB.2, -OUTPUT.2
- net GND: now also -OUTPUT.1, C4.2, C6.+, C7.+, ON-.A, R3.2, R3.3, R4.2, R4.3, R7.1; no longer Q1.E, R2.2, R2.3
- net N$1: now also C7.-, D5.C, R2.1, R4.1, VADJ1.1; no longer IADJ.2, R3.1, R3.2, R4.2
- net N$2: now also +INPUT.2, SW_P.2; no longer R4.1, R5.2
- net N$3: now also R3.1; no longer R2.1
- net N$4: now also ON-.C, R8.2; no longer Q1.C, R7.1
- net N$5: now also -INPUT.1, SW_N.2; no longer R5.1, R6.2
- net V-: now also C4.1, D4.A, R8.1, SW_N.1, VADJ1.3; no longer -INPUT.1
- net VCC: now also C1.1, D2.C, SW_P.1, VADJ.3; no longer +INPUT.2, VIN_SEL.1, VIN_SEL.3
Routing:
- net VADJ_IN: track 83.4 -> 0.00 mm
- net VOUT: track 61.5 -> 0.00 mm
- net +VOUT: track 0.00 -> 59.4 mm
- net N$1: track 41.8 -> 0.00 mm, vias 1 -> 0
- net VCC: track 97.4 -> 129.0 mm
- net IADJ_IN: track 29.5 -> 0.00 mm
- net N$8: track 16.7 -> 0.00 mm
- net N$4: track 10.5 -> 0.00 mm
- net GND: track 0.00 -> 9.09 mm
- net N$5: track 5.05 -> 0.00 mm
- net N$2: track 4.86 -> 0.00 mm
- net N$3: track 59.8 -> 56.0 mm
